File: Motorpro/MotorProRePro.brd (EAGLE design)
At the start: 100 x 80 mm, 19 parts, among them IC1 7805T, Q1 BTA06-600BRG

Commit message: Board modificada
Parts:
- moved R1 101.8 mm to (74.9, 91.4), turned to 180 degrees
- moved R4 77.5 mm to (15.2, 53.3)
- moved PINES 76.2 mm to (17.8, 94.0)
- moved R6 66.1 mm to (55.9, 92.7)
- moved IC1 63.9 mm to (34.3, 34.3), turned to 180 degrees
- moved C2 47.1 mm to (50.8, 49.5), turned to 180 degrees
- moved ARDUINO_NANO1 44.5 mm to (27.9, 78.7)
- moved VCC_12V 44.4 mm to (12.7, 43.2), turned to 0 degrees
- moved R5 39.9 mm to (33.0, 53.3)
- moved POTENCIA 31.9 mm to (88.9, 6.35), turned to 180 degrees
- moved R3 30.5 mm to (85.1, 20.3)
- moved Q1 29.0 mm to (71.1, 41.9)
- moved CERO 28.0 mm to (57.1, 33.0)
- moved OK1 24.1 mm to (72.4, 55.9), turned to 270 degrees
- moved C1 21.7 mm to (43.2, 61.0), turned to 180 degrees
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Routing:
- net REFERENCIA: track 31.5 -> 105.2 mm
- net N$13: track 66.9 -> 7.62 mm
- net VCC: track 111.7 -> 154.1 mm
- net N$8: track 50.7 -> 11.4 mm
- net GND: track 220.0 -> 183.2 mm
- net N$14: track 11.5 -> 46.0 mm
- net N$5: track 48.9 -> 17.9 mm
- net N$1: track 43.7 -> 69.9 mm
- net FASE: track 68.4 -> 93.9 mm
- net ZERO: track 169.0 -> 149.1 mm
- net N$4: track 13.2 -> 33.0 mm
- net N$9: track 25.7 -> 7.62 mm
- net N$12: track 25.7 -> 7.62 mm
- net N$11: track 25.7 -> 7.62 mm
- net N$10: track 25.7 -> 7.62 mm
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Other:
- board size 100 x 80 mm -> 106.7 x 102.5 mm

Commit message: Para eviar a china
Parts:
- added IC2: LF353N, linear:DIL08
- added R10, R11: 1k, rcl:0207/10
- added R8: 410, rcl:0207/10
- added R9: 10k, rcl:0207/10
- added T1: 2N3904, transistor:TO92
Connections:
- new net N$16: R8.2, T1.2
- new net N$17: IC2.3, R9.1, T1.3
- new net N$18: IC2.2, R10.2, R11.1
- new net V+: IC2.8
- new net V-: IC2.4
- net GND: now also R10.1, T1.1
- net VCC: now also R11.2, R9.2
- net ZERO: now also IC2.1, R8.1
Changed lines of the file:
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@@
 <attribute name="VALUE" x="5.1054" y="33.655" size="1.778" layer="27" ratio="10"/>
+</element>
+<element name="R8" library="rcl" library_urn="urn:adsk.eagle:library:334" package="0207/10" package3d_urn="urn:adsk.eagle:package:23491/2" value="410" x="3.81" y="-6.35" smashed="yes">
+<attribute name="NAME" x="0.762" y="-4.826" size="1.27" layer="25" ratio="10"/>
+<attribute name="POPULARITY" value="36" x="3.81" y="-6.35" size="1.778" layer="27" display="off"/>
+<attribute name="SPICEPREFIX" value="R" x="3.81" y="-6.35" size="1.778" layer="27" display="off"/>
+<attribute name="VALUE" x="1.5494" y="-6.985" size="1.27" layer="27" ratio="10"/>
+</element>
+<element name="T1" library="transistor" library_urn="urn:adsk.eagle:library:402" package="TO92" package3d_urn="urn:adsk.eagle:package:28523/2" value="2N3904" x="1.27" y="-11.43" smashed="yes">
+<attribute name="NAME" x="4.445" y="-10.795" size="1.27" layer="25" ratio="10"/>
+<attribute name="POPULARITY" value="27" x="1.27" y="-11.43" size="1.778" layer="27" display="off"/>
+<attribute name="VALUE" x="4.445" y="-12.7" size="1.27" layer="27" ratio="10"/>
+</element>
+<element name="R9" library="rcl" library_urn="urn:adsk.eagle:library:334" package="0207/10" package3d_urn="urn:adsk.eagle:package:23491/2" value="10k" x="3.81" y="-17.78" smashed="yes">
+<attribute name="NAME" x="0.762" y="-16.256" size="1.27" layer="25" ratio="10"/>
+<attribute name="POPULARITY" value="36" x="3.81" y="-17.78" size="1.778" layer="27" display="off"/>
+<attribute name="SPICEPREFIX" value="R" x="3.81" y="-17.78" size="1.778" layer="27" display="off"/>
+<attribute name="VALUE" x="1.5494" y="-18.415" size="1.27" layer="27" ratio="10"/>
+</element>
+<element name="IC2" library="linear" library_urn="urn:adsk.eagle:library:262" package="DIL08" package3d_urn="urn:adsk.eagle:package:16409/2" value="LF353N" x="5.08" y="-24.13" smashed="yes">
+<attribute name="NAME" x="-0.254" y="-27.051" size="1.27" layer="25" ratio="10" rot="R90"/>
+<attribute name="POPULARITY" value="0" x="5.08" y="-24.13" size="1.778" layer="27" display="off"/>
+<attribute name="VALUE" x="1.524" y="-24.765" size="1.27" layer="27" ratio="10"/>
+</element>
+<element name="R10" library="rcl" library_urn="urn:adsk.eagle:library:334" package="0207/10" package3d_urn="urn:adsk.eagle:package:23491/2" value="1k" x="3.81" y="-33.02" smashed="yes">
+<attribute name="NAME" x="0.762" y="-31.496" size="1.27" layer="25" ratio="10"/>
+<attribute name="POPULARITY" value="36" x="3.81" y="-33.02" size="1.778" layer="27" display="off"/>
+<attribute name="SPICEPREFIX" value="R" x="3.81" y="-33.02" size="1.778" layer="27" display="off"/>
+<attribute name="VALUE" x="1.5494" y="-33.655" size="1.27" layer="27" ratio="10"/>
+</element>
+<element name="R11" library="rcl" library_urn="urn:adsk.eagle:library:334" package="0207/10" package3d_urn="urn:adsk.eagle:package:23491/2" value="1k" x="3.81" y="-38.1" smashed="yes">
+<attribute name="NAME" x="0.762" y="-36.576" size="1.27" layer="25" ratio="10"/>
+<attribute name="POPULARITY" value="36" x="3.81" y="-38.1" size="1.778" layer="27" display="off"/>
+<attribute name="SPICEPREFIX" value="R" x="3.81" y="-38.1" size="1.778" layer="27" display="off"/>
+<attribute name="VALUE" x="1.5494" y="-38.735" size="1.27" layer="27" ratio="10"/>
 </element>
 </elements>
@@
 <wire x1="34.29" y1="44.45" x2="34.29" y2="41.91" width="0.762" layer="16"/>
 <wire x1="40.64" y1="60.96" x2="26.67" y2="60.96" width="0.762" layer="1"/>
+<contactref element="T1" pad="1"/>
+<contactref element="R10" pad="1"/>
+<wire x1="2.54" y1="-11.43" x2="17.7038" y2="43.18" width="0" layer="19" extent="1-1"/>
+<wire x1="-1.27" y1="-33.02" x2="2.54" y2="-11.43" width="0" layer="19" extent="1-1"/>
 </signal>
 <signal name="5V">
@@
 <wire x1="53.34" y1="73.66" x2="43.18" y2="73.66" width="0.762" layer="16"/>
 <wire x1="53.34" y1="49.53" x2="53.34" y2="73.66" width="0.762" layer="16"/>
+<contactref element="R9" pad="2"/>
+<contactref element="R11" pad="2"/>
+<wire x1="31.75" y1="44.45" x2="28.575" y2="48.895" width="0" layer="19" extent="1-1"/>
+<wire x1="8.89" y1="-17.78" x2="31.75" y2="44.45" width="0" layer="19" extent="1-1"/>
+<wire x1="8.89" y1="-38.1" x2="8.89" y2="-17.78" width="0" layer="19" extent="1-1"/>
 </signal>
 <signal name="REFERENCIA">
@@
 <wire x1="23.495" y1="33.02" x2="23.495" y2="53.34" width="0.762" layer="16"/>
 <wire x1="53.34" y1="33.02" x2="23.495" y2="33.02" width="0.762" layer="16"/>
+<contactref element="R8" pad="1"/>
+<contactref element="IC2" pad="1"/>
+<wire x1="-1.27" y1="-6.35" x2="20.32" y2="53.34" width="0" layer="19" extent="1-1"/>
+<wire x1="1.27" y1="-27.94" x2="-1.27" y2="-6.35" width="0" layer="19" extent="1-1"/>
 </signal>
 <signal name="SALIDA">
@@
 <wire x1="10.16" y1="93.98" x2="2.54" y2="93.98" width="0.762" layer="1"/>
 </signal>
+<signal name="N$16">
+<contactref element="R8" pad="2"/>
+<contactref element="T1" pad="2"/>
+<wire x1="8.89" y1="-6.35" x2="1.27" y2="-9.525" width="0" layer="19" extent="1-1"/>
+</signal>
+<signal name="N$17">
+<contactref element="T1" pad="3"/>
+<contactref element="R9" pad="1"/>
+<contactref element="IC2" pad="3"/>
+<wire x1="-1.27" y1="-17.78" x2="6.35" y2="-27.94" width="0" layer="19" extent="1-1"/>
+<wire x1="0" y1="-11.43" x2="-1.27" y2="-17.78" width="0" layer="19" extent="1-1"/>
+</signal>
+<signal name="V+">
+<contactref element="IC2" pad="8"/>
+</signal>
+<signal name="V-">
+<contactref element="IC2" pad="4"/>
+</signal>
+<signal name="N$18">
+<contactref element="R11" pad="1"/>
+<contactref element="R10" pad="2"/>
+<contactref element="IC2" pad="2"/>
+<wire x1="8.89" y1="-33.02" x2="-1.27" y2="-38.1" width="0" layer="19" extent="1-1"/>
+<wire x1="3.81" y1="-27.94" x2="8.89" y2="-33.02" width="0" layer="19" extent="1-1"/>
+</signal>
 </signals>

Commit message: avance pcb y codigo final
Parts:
- removed Q1: BTA06-600BRG, BTA06-600BRG:TO254P1040X460X1975-3
- added U1: BTA41-600BRG, BTA41-600BRG:TO552P460X1530X2985-3P
Connections:
- net FASE: now also U1.2; no longer Q1.2
- net N$7: now also U1.1; no longer Q1.1
- net N$8: now also U1.3; no longer Q1.3
Routing:
- net FASE: track 93.9 -> 77.4 mm
- net N$7: track 33.3 -> 18.7 mm
- net N$8: track 11.4 -> 0.00 mm
Changed lines of the file:
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@@
 <attribute name="VALUE" x="96.4946" y="15.875" size="1.778" layer="27" ratio="10" rot="R180"/>
-</element>
-<element name="Q1" library="BTA06-600BRG" package="TO254P1040X460X1975-3" value="BTA06-600BRG" x="71.12" y="41.91" smashed="yes">
-<attribute name="AVAILABILITY" value="Unavailable" x="120.65" y="-20.32" size="1.778" layer="27" display="off"/>
-<attribute name="DESCRIPTION" value=" BTA06 Series 600 Vdrm 6 A Flange Mount Standard Triac Thyristor - TO-220AB " x="120.65" y="-20.32" size="1.778" layer="27" display="off"/>
-<attribute name="MF" value="STMicroelectronics" x="120.65" y="-20.32" size="1.778" layer="27" display="off"/>
-<attribute name="MP" value="BTA06-600BRG" x="120.65" y="-20.32" size="1.778" layer="27" display="off"/>
-<attribute name="NAME" x="68.2146" y="44.8154" size="1.27236875" layer="25"/>
-<attribute name="PACKAGE" value="TO-220 STMicroelectronics" x="120.65" y="-20.32" size="1.778" layer="27" display="off"/>
-<attribute name="PRICE" value="None" x="120.65" y="-20.32" size="1.778" layer="27" display="off"/>
-<attribute name="VALUE" x="68.114290625" y="38.30315" size="1.27241875" layer="27"/>
 </element>
 <element name="R1" library="pot" library_urn="urn:adsk.eagle:library:331" package="3RP/1610N" package3d_urn="urn:adsk.eagle:package:22726/1" value="" x="74.93" y="91.44" smashed="yes" rot="R180">
@@
 <attribute name="SPICEPREFIX" value="R" x="3.81" y="-38.1" size="1.778" layer="27" display="off"/>
 <attribute name="VALUE" x="1.5494" y="-38.735" size="1.27" layer="27" ratio="10"/>
+</element>
+<element name="U1" library="BTA41-600BRG" package="TO552P460X1530X2985-3P" value="BTA41-600BRG" x="2.54" y="-43.18" smashed="yes">
+<attribute name="ALLIED_NUMBER" value="70332160" x="2.54" y="-43.18" size="1.778" layer="27" display="off"/>
+<attribute name="DESCRIPTION" value="TRIAC BTA41-600BRG, 600V, Gate Trigger 1.3V 100mA, TOP Insulated 3-Pin" x="2.54" y="-43.18" size="1.778" layer="27" display="off"/>
+<attribute name="HEIGHT" value="4.6mm" x="2.54" y="-43.18" size="1.778" layer="27" display="off"/>
+<attribute name="MANUFACTURER_NAME" value="STMicroelectronics" x="2.54" y="-43.18" size="1.778" layer="27" display="off"/>
+<attribute name="MANUFACTURER_PART_NUMBER" value="BTA41-600BRG" x="2.54" y="-43.18" size="1.778" layer="27" display="off"/>
+<attribute name="NAME" x="2.54" y="-43.18" size="1.27" layer="25" align="center"/>
+<attribute name="RS_PART_NUMBER" value="6871007P" x="2.54" y="-43.18" size="1.778" layer="27" display="off"/>
+<attribute name="RS_PRICE-STOCK" value="http://uk.rs-online.com/web/p/products/6871007P" x="2.54" y="-43.18" size="1.778" layer="27" display="off"/>
+<attribute name="VALUE" x="2.54" y="-43.18" size="1.27" layer="27" align="center"/>
 </element>
 </elements>
@@
 <contactref element="R3" pad="2"/>
 <contactref element="R7" pad="2"/>
-<contactref element="Q1" pad="2"/>
 <wire x1="99.695" y1="20.32" x2="90.17" y2="20.32" width="0.762" layer="16"/>
 <wire x1="93.9038" y1="6.35" x2="99.695" y2="6.35" width="0.762" layer="16"/>
@@
 <wire x1="91.44" y1="49.53" x2="90.805" y2="48.895" width="0.762" layer="1"/>
 <wire x1="74.295" y1="48.895" x2="90.805" y2="48.895" width="0.762" layer="1"/>
-<wire x1="73.66" y1="41.91" x2="73.66" y2="48.26" width="0.762" layer="1"/>
 <wire x1="74.295" y1="48.895" x2="73.66" y2="48.26" width="0.762" layer="1"/>
 <wire x1="89.746665625" y1="22.436665625" x2="89.746665625" y2="20.743334375" width="0.762" layer="16"/>
 <wire x1="90.17" y1="20.32" x2="89.746665625" y2="20.743334375" width="0.762" layer="16"/>
 <wire x1="89.746665625" y1="22.436665625" x2="73.66" y2="31.75" width="0.762" layer="16"/>
-<wire x1="73.66" y1="31.75" x2="73.66" y2="41.91" width="0.762" layer="16"/>
+<contactref element="U1" pad="2"/>
+<wire x1="73.66" y1="31.75" x2="73.66" y2="48.26" width="0" layer="19" extent="1-16"/>
+<wire x1="8.065" y1="-43.18" x2="93.9038" y2="6.35" width="0" layer="19" extent="1-1"/>
 </signal>
 <signal name="NEUTRO">
@@
 <signal name="N$8">
 <contactref element="OK1" pad="4"/>
-<contactref element="Q1" pad="3"/>
-<wire x1="76.2" y1="41.91" x2="76.2" y2="53.34" width="0.762" layer="16"/>
+<contactref element="U1" pad="3"/>
+<wire x1="13.59" y1="-43.18" x2="76.2" y2="53.34" width="0" layer="19" extent="1-1"/>
 </signal>
 <signal name="N$7">
-<contactref element="Q1" pad="1"/>
 <contactref element="MOTOR" pad="3"/>
-<wire x1="71.12" y1="27.305" x2="71.12" y2="41.91" width="0.762" layer="16"/>
 <wire x1="74.8538" y1="10.16" x2="74.8538" y2="23.5712" width="0.762" layer="16"/>
 <wire x1="74.8538" y1="23.5712" x2="71.12" y2="27.305" width="0.762" layer="16"/>
+<contactref element="U1" pad="1"/>
+<wire x1="2.54" y1="-43.18" x2="74.8538" y2="10.16" width="0" layer="19" extent="1-1"/>
 </signal>
 <signal name="N$9">
