File: Motorpro/MotorProRePro.sch (EAGLE design)
At the start: 25 parts, among them IC1 7805T, IC2 LF353N, Q1 BTA06-600BRG, T1 2N3904

Commit message: avance pcb y codigo final
Parts:
- removed Q1: BTA06-600BRG, BTA06-600BRG:BTA06-600BRG
- added U1: BTA41-600BRG, BTA41-600BRG:BTA41-600BRG
Connections:
- net FASE: now also U1.A2; no longer Q1.A2
- net N$7: now also U1.A1; no longer Q1.A1
- net N$8: now also U1.G; no longer Q1.G
Changed lines of the file:
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@@
 <part name="R6" library="rcl" library_urn="urn:adsk.eagle:library:334" deviceset="R-US_" device="0207/10" package3d_urn="urn:adsk.eagle:package:23491/2" value="330"/>
 <part name="R7" library="rcl" library_urn="urn:adsk.eagle:library:334" deviceset="R-US_" device="0207/10" package3d_urn="urn:adsk.eagle:package:23491/2" value="180"/>
-<part name="Q1" library="BTA06-600BRG" deviceset="BTA06-600BRG" device=""/>
 <part name="MOTOR" library="con-ptr500" library_urn="urn:adsk.eagle:library:181" deviceset="AK500/3-H" device="" package3d_urn="urn:adsk.eagle:package:9899/1"/>
 <part name="PINES" library="con-lstb" library_urn="urn:adsk.eagle:library:162" deviceset="MA07-1" device="" package3d_urn="urn:adsk.eagle:package:8341/1"/>
@@
 <part name="R10" library="rcl" library_urn="urn:adsk.eagle:library:334" deviceset="R-US_" device="0207/10" package3d_urn="urn:adsk.eagle:package:23491/2" value="1k"/>
 <part name="R11" library="rcl" library_urn="urn:adsk.eagle:library:334" deviceset="R-US_" device="0207/10" package3d_urn="urn:adsk.eagle:package:23491/2" value="1k"/>
+<part name="U1" library="BTA41-600BRG" deviceset="BTA41-600BRG" device=""/>
 </parts>
 <sheets>
@@
 <attribute name="VALUE" x="100.33" y="-13.462" size="1.778" layer="96"/>
 </instance>
-<instance part="Q1" gate="G$1" x="134.62" y="-17.78" smashed="yes">
-<attribute name="NAME" x="123.1896" y="-12.69981875" size="1.778059375" layer="95"/>
-<attribute name="VALUE" x="123.177" y="-22.865790625" size="1.78003125" layer="96"/>
-</instance>
 <instance part="MOTOR" gate="-1" x="139.7" y="20.32" smashed="yes">
 <attribute name="NAME" x="138.43" y="21.209" size="1.778" layer="95" rot="R180"/>
@@
 <attribute name="NAME" x="-19.2786" y="16.51" size="1.778" layer="95" rot="R90"/>
 <attribute name="VALUE" x="-14.478" y="16.51" size="1.778" layer="96" rot="R90"/>
+</instance>
+<instance part="U1" gate="G$1" x="127" y="-33.02" smashed="yes">
+<attribute name="NAME" x="146.05" y="-25.4" size="1.778" layer="95" align="center-left"/>
+<attribute name="VALUE" x="146.05" y="-27.94" size="1.778" layer="96" align="center-left"/>
 </instance>
 </instances>
@@
 </segment>
 <segment>
-<wire x1="134.62" y1="-12.7" x2="134.62" y2="-10.16" width="0.1524" layer="91"/>
 <pinref part="R7" gate="G$1" pin="2"/>
-<wire x1="134.62" y1="-10.16" x2="109.22" y2="-10.16" width="0.1524" layer="91"/>
+<wire x1="139.7" y1="-10.16" x2="124.46" y2="-10.16" width="0.1524" layer="91"/>
 <label x="139.7" y="-10.16" size="1.778" layer="95" xref="yes"/>
-<wire x1="139.7" y1="-10.16" x2="134.62" y2="-10.16" width="0.1524" layer="91"/>
-<junction x="134.62" y="-10.16"/>
-<pinref part="Q1" gate="G$1" pin="A2"/>
+<wire x1="124.46" y1="-10.16" x2="109.22" y2="-10.16" width="0.1524" layer="91"/>
+<pinref part="U1" gate="G$1" pin="A2"/>
+<wire x1="127" y1="-35.56" x2="124.46" y2="-35.56" width="0.1524" layer="91"/>
+<wire x1="124.46" y1="-35.56" x2="124.46" y2="-10.16" width="0.1524" layer="91"/>
+<junction x="124.46" y="-10.16"/>
 </segment>
 </net>
@@
 <net name="N$8" class="0">
 <segment>
-<wire x1="129.54" y1="-17.78" x2="109.22" y2="-17.78" width="0.1524" layer="91"/>
+<wire x1="121.92" y1="-17.78" x2="109.22" y2="-17.78" width="0.1524" layer="91"/>
 <wire x1="109.22" y1="-17.78" x2="109.22" y2="-20.32" width="0.1524" layer="91"/>
 <pinref part="OK1" gate="-1" pin="A1"/>
 <wire x1="109.22" y1="-20.32" x2="88.9" y2="-20.32" width="0.1524" layer="91"/>
-<pinref part="Q1" gate="G$1" pin="G"/>
+<pinref part="U1" gate="G$1" pin="G"/>
+<wire x1="149.86" y1="-33.02" x2="149.86" y2="-25.4" width="0.1524" layer="91"/>
+<wire x1="149.86" y1="-25.4" x2="121.92" y2="-25.4" width="0.1524" layer="91"/>
+<wire x1="121.92" y1="-25.4" x2="121.92" y2="-17.78" width="0.1524" layer="91"/>
 </segment>
 </net>
 <net name="N$7" class="0">
 <segment>
-<pinref part="Q1" gate="G$1" pin="A1"/>
-<wire x1="134.62" y1="-20.32" x2="157.48" y2="-20.32" width="0.1524" layer="91"/>
+<wire x1="127" y1="-20.32" x2="157.48" y2="-20.32" width="0.1524" layer="91"/>
 <wire x1="157.48" y1="-20.32" x2="157.48" y2="12.7" width="0.1524" layer="91"/>
 <wire x1="157.48" y1="12.7" x2="152.4" y2="12.7" width="0.1524" layer="91"/>
@@
 <wire x1="152.4" y1="12.7" x2="152.4" y2="10.16" width="0.1524" layer="91"/>
 <wire x1="152.4" y1="10.16" x2="144.78" y2="10.16" width="0.1524" layer="91"/>
-</segment>
-</net>
+<pinref part="U1" gate="G$1" pin="A1"/>
+<wire x1="127" y1="-33.02" x2="127" y2="-20.32" width="0.1524" layer="91"/>
+</segment>
+</net>
